File: access_control.kicad_sch (KiCad schematic)
At the start: 78 parts, among them J1 Conn_01x04_Pin, J10 Screw_Terminal_01x02, J2 Screw_Terminal_01x04, J3 Screw_Terminal_01x04, J4 Screw_Terminal_01x02, J5 Screw_Terminal_01x04, J6 Screw_Terminal_01x04, J7 Screw_Terminal_01x02, J8 Screw_Terminal_01x02, J9 Screw_Terminal_01x02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

Commit message: Finilized editing PCB, generated BOM and grb files. PCB files are sent to JLCPCB
Parts:
- removed Q1, Q2, Q3, Q4: NMOS, Package_TO_SOT_SMD:SOT-23_Handsoldering, symbol Simulation_SPICE:NMOS
- added Q1, Q2, Q3, Q4: FDV305N, Package_TO_SOT_SMD:SOT-23, symbol Transistor_FET:DMG2301L
- R10, R11, R12, R13: LCSC (none) -> C2907256
- R2, R3: LCSC (none) -> C2907326
- R9: LCSC (none) -> C2907295
Connections:
- net DOOR1_DRAIN: now also Q1.3 (D)
- net DOOR2_DRAIN: now also Q2.3 (D)
- net DOOR3_DRAIN: now also Q3.3 (D)
- net DOOR4_DRAIN: now also Q4.3 (D)
- net GND: now also Q1.2 (S), Q2.2 (S), Q3.2 (S), Q4.2 (S)
- net at R11.2, R4.2: now also Q1.1 (G)
- net at R10.2, R5.2: now also Q2.1 (G)
- net at R12.2, R7.2: now also Q4.1 (G)
- net at R13.2, R6.2: now also Q3.1 (G)
